File: board/BLE_PP_v16.brd (EAGLE design)
At the start: 27.7 x 28.4 mm, 18 parts, among them SW4 SW_SLIDECUS12B, U1 MOD_CYBLE014008-00, U2 REG_TPS61221

Commit message: スリープに入るアルゴリズム＆L2CAP paramUpdateRequestを送るアルゴリズムを変更。SleepからIDボタンで復帰。マニュアルの修正。
Parts:
- R2: value 560k -> 390k
- R3: value 200k -> 100k
Changed lines of the file:
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@@
 <?xml version="1.0" encoding="utf-8"?>
 <!DOCTYPE eagle SYSTEM "eagle.dtd">
-<eagle version="8.1.0">
+<eagle version="7.7.0">
 <drawing>
 <settings>
@@
 <setting verticaltext="up"/>
 </settings>
-<grid distance="1" unitdist="mm" unit="mm" style="lines" multiple="1" display="yes" altdistance="0.1" altunitdist="mm" altunit="mm"/>
+<grid distance="1.27" unitdist="mm" unit="mm" style="lines" multiple="1" display="yes" altdistance="0.1" altunitdist="mm" altunit="mm"/>
 <layers>
 <layer number="1" name="Top" color="4" fill="1" visible="no" active="yes"/>
@@
 </element>
 <element name="SW6" library="akita" package="SW_EVQP7" value="" x="5.7" y="15" rot="MR270"/>
-<element name="R2" library="akita" package="0603" value="560k" x="13" y="23" smashed="yes" rot="R180">
+<element name="R2" library="akita" package="0603" value="390k" x="13" y="23" smashed="yes" rot="R180">
 <attribute name="NAME" x="13.789" y="22.303" size="0.8128" layer="25" font="vector" rot="R180"/>
 <attribute name="VALUE" x="14.016" y="24.778" size="0.8128" layer="27" font="vector" rot="R180"/>
 </element>
-<element name="R3" library="akita" package="0603" value="200k" x="17" y="23" smashed="yes" rot="R180">
+<element name="R3" library="akita" package="0603" value="100k" x="17" y="23" smashed="yes" rot="R180">
 <attribute name="NAME" x="17.689" y="22.203" size="0.8128" layer="25" font="vector" rot="R180"/>
 <attribute name="VALUE" x="18.016" y="24.778" size="0.8128" layer="27" font="vector" rot="R180"/>
